File: keyb_left/kai_split_left.kicad_sch (KiCad schematic)
At the start: 70 parts, among them J1 USB_C_Receptacle_USB2.0, SW1 SW_Push, U2 ATmega32U4-A, Y1 16MHz

Commit message: added another library
Parts:
- added J2: AudioJack4, symbol Connector_Audio:AudioJack4
- added R10, R9: 1k, symbol Device:R_Small
Connections:
- net +5V: now also J2.T
- net GND: now also J2.S
- net RX: now reaches U2.20 (PD2)
- net RX: now also R9.2
- net TX: now reaches U2.21 (PD3)
- net TX: now also R10.2
- new net: J2.R2, R9.1
- new net: J2.R1, R10.1
Other:
- moved on the sheet: C2, C3, C4, C5

Commit message: routing finsihed, very poorly
Parts:
- removed R2, R3: 22, symbol Device:R_Small
- C1, C2, C3, C4, C5, C6, C7: footprint (none) -> Capacitor_SMD:C_0805_2012Metric
- D1, D10, D11, D12, D13, D14, D15, D16, D17, D18, D19, D2, D20, D21, D22, D23, D24, D25: footprint (none) -> Diode_SMD:D_SOD-123
- D3: renamed from D5; footprint (none) -> Diode_SMD:D_SOD-123
- D4: renamed from D7; footprint (none) -> Diode_SMD:D_SOD-123
- D5: renamed from D9; footprint (none) -> Diode_SMD:D_SOD-123
- D6: renamed from D3; footprint (none) -> Diode_SMD:D_SOD-123
- D7: renamed from D4; footprint (none) -> Diode_SMD:D_SOD-123
- D8: renamed from D6; footprint (none) -> Diode_SMD:D_SOD-123
- D9: renamed from D8; footprint (none) -> Diode_SMD:D_SOD-123
- F1: footprint (none) -> Fuse:Fuse_1206_3216Metric
- J1: footprint (none) -> Connector_USB:USB_C_Receptacle_Amphenol_12401610E4-2A
- J2: footprint (none) -> Keebio-Parts:TRRS-PJ-320A
- MX1, MX10, MX11, MX12, MX13, MX14, MX15, MX16, MX17, MX18, MX19, MX2, MX20, MX21, MX22, MX23, MX24, MX25: footprint (none) -> MX_Alps_Hybrid:MX-1U-NoLED
- MX3: renamed from MX5; footprint (none) -> MX_Alps_Hybrid:MX-1U-NoLED
- MX4: renamed from MX7; footprint (none) -> MX_Alps_Hybrid:MX-1U-NoLED
- MX5: renamed from MX9; footprint (none) -> MX_Alps_Hybrid:MX-1U-NoLED
- MX6: renamed from MX3; footprint (none) -> MX_Alps_Hybrid:MX-1U-NoLED
- MX7: renamed from MX4; footprint (none) -> MX_Alps_Hybrid:MX-1U-NoLED
- MX8: renamed from MX6; footprint (none) -> MX_Alps_Hybrid:MX-1U-NoLED
- MX9: renamed from MX8; footprint (none) -> MX_Alps_Hybrid:MX-1U-NoLED
- R1, R10, R4, R5, R6, R7, R8, R9: footprint (none) -> Resistor_SMD:R_0805_2012Metric
- SW1: footprint (none) -> random-keyboard-parts:SKQG-1155865
- Y1: footprint (none) -> Crystal:Crystal_SMD_3225-4Pin_3.2x2.5mm
Connections:
- net COL0: now also U2.25 (PD4)
- net COL1: now also U2.26 (PD6)
- net COL2: now also U2.27 (PD7)
- net COL3: now also U2.28 (PB4); no longer MX19.1 (COL)
- net COL4: now also U2.29 (PB5)
- net D+: now also U2.4 (D+)
- net D-: now also U2.3 (D-)
- net ROW0: now also U2.37 (PF6)
- net ROW1: now also U2.38 (PF5)
- net ROW2: now also U2.39 (PF4)
- net ROW3: now also U2.40 (PF1)
- net ROW4: now also U2.41 (PF0)
- net at D19.2 (A): no longer MX19.2 (ROW)
Other:
- moved on the sheet: MX19, R1
